Commit message: improve and fix small bugs / uncertainties

File: urdf/rover.urdf.xacro (robot description, xacro)
@@ -33,46 +33,36 @@
     </inertial>
   </link>
-  <link name="left_wheel">
-    <visual>
-      <origin rpy="1.5708 0 0"/>
-      <geometry><cylinder radius="${wheel_radius}" length="${wheel_width}"/></geometry>
-    </visual>
-    <collision>
-      <origin rpy="1.5708 0 0"/>
-      <geometry><cylinder radius="${wheel_radius}" length="${wheel_width}"/></geometry>
-    </collision>
-    <inertial>
-      <mass value="0.25"/>
-      <origin xyz="0 0 0"/>
-      <inertia ixx="0.0003" ixy="0" ixz="0" iyy="0.0003" iyz="0" izz="0.0005"/>
-    </inertial>
-  </link>
-  <link name="right_wheel">
-    <visual>
-      <origin rpy="1.5708 0 0"/>
-      <geometry><cylinder radius="${wheel_radius}" length="${wheel_width}"/></geometry>
-    </visual>
-    <collision>
-      <origin rpy="1.5708 0 0"/>
-      <geometry><cylinder radius="${wheel_radius}" length="${wheel_width}"/></geometry>
-    </collision>
-    <inertial>
-      <mass value="0.25"/>
-      <origin xyz="0 0 0"/>
-      <inertia ixx="0.0003" ixy="0" ixz="0" iyy="0.0003" iyz="0" izz="0.0005"/>
-    </inertial>
-  </link>
-  <joint name="left_wheel_joint" type="continuous">
-    <parent link="base_link"/>
-    <child link="left_wheel"/>
-    <origin xyz="0 ${base_width / 2.0} -0.04" rpy="0 0 0"/>
-    <axis xyz="0 1 0"/>
-  </joint>
-  <joint name="right_wheel_joint" type="continuous">
-    <parent link="base_link"/>
-    <child link="right_wheel"/>
-    <origin xyz="0 ${-base_width / 2.0} -0.04" rpy="0 0 0"/>
-    <axis xyz="0 1 0"/>
-  </joint>
+  <xacro:macro name="wheel" params="name x y">
+    <link name="${name}_wheel">
+      <visual>
+        <origin rpy="1.5708 0 0"/>
+        <geometry><cylinder radius="${wheel_radius}" length="${wheel_width}"/></geometry>
+      </visual>
+      <collision>
+        <origin rpy="1.5708 0 0"/>
+        <geometry><cylinder radius="${wheel_radius}" length="${wheel_width}"/></geometry>
+      </collision>
+      <inertial>
+        <mass value="0.25"/>
+        <origin xyz="0 0 0"/>
+        <inertia ixx="0.0003" ixy="0" ixz="0" iyy="0.0003" iyz="0" izz="0.0005"/>
+      </inertial>
+    </link>
+    <joint name="${name}_wheel_joint" type="continuous">
+      <parent link="base_link"/>
+      <child link="${name}_wheel"/>
+      <origin xyz="${x} ${y} -0.04" rpy="0 0 0"/>
+      <axis xyz="0 1 0"/>
+    </joint>
+    <gazebo reference="${name}_wheel">
+      <material>Gazebo/Black</material>
+      <mu1>1.0</mu1>
+      <mu2>1.0</mu2>
+    </gazebo>
+  </xacro:macro>
+  <xacro:wheel name="left_front" x="${base_length * 0.32}" y="${base_width / 2.0}"/>
+  <xacro:wheel name="left_rear" x="${-base_length * 0.32}" y="${base_width / 2.0}"/>
+  <xacro:wheel name="right_front" x="${base_length * 0.32}" y="${-base_width / 2.0}"/>
+  <xacro:wheel name="right_rear" x="${-base_length * 0.32}" y="${-base_width / 2.0}"/>
   <link name="lidar_link">
     <visual>
@@ -96,14 +86,4 @@
     <material>Gazebo/Green</material>
   </gazebo>
-  <gazebo reference="left_wheel">
-    <material>Gazebo/Black</material>
-    <mu1>1.0</mu1>
-    <mu2>1.0</mu2>
-  </gazebo>
-  <gazebo reference="right_wheel">
-    <material>Gazebo/Black</material>
-    <mu1>1.0</mu1>
-    <mu2>1.0</mu2>
-  </gazebo>
   <gazebo reference="lidar_link">
     <material>Gazebo/Black</material>
@@ -124,5 +104,5 @@
         <range>
           <min>0.08</min>
-          <max>6.0</max>
+          <max>12.0</max>
           <resolution>0.01</resolution>
         </range>
@@ -132,14 +112,26 @@
   <gazebo>
     <plugin filename="gz-sim-diff-drive-system" name="gz::sim::systems::DiffDrive">
-      <left_joint>left_wheel_joint</left_joint>
-      <right_joint>right_wheel_joint</right_joint>
+      <left_joint>left_front_wheel_joint</left_joint>
+      <left_joint>left_rear_wheel_joint</left_joint>
+      <right_joint>right_front_wheel_joint</right_joint>
+      <right_joint>right_rear_wheel_joint</right_joint>
       <wheel_separation>${wheel_separation}</wheel_separation>
       <wheel_radius>${wheel_radius}</wheel_radius>
       <topic>/cmd_vel</topic>
-      <odom_topic>/odom</odom_topic>
+      <odom_topic>/wheel_odom</odom_topic>
       <frame_id>odom</frame_id>
       <child_frame_id>base_footprint</child_frame_id>
       <odom_publish_frequency>30</odom_publish_frequency>
     </plugin>
+    <!-- Simulation truth: unlike wheel integration, this follows the model's
+         physical pose even when four-wheel skid steering slips. -->
+    <plugin filename="gz-sim-odometry-publisher-system"
+            name="gz::sim::systems::OdometryPublisher">
+      <odom_topic>/odom</odom_topic>
+      <odom_frame>odom</odom_frame>
+      <robot_base_frame>base_footprint</robot_base_frame>
+      <dimensions>2</dimensions>
+      <odom_publish_frequency>30</odom_publish_frequency>
+    </plugin>
   </gazebo>
 </robot>
